Commit message: Update phantomX_model.xacro

File: hexapod_description/urdf/phantomX_model.xacro (robot description, xacro)
@@ -85,5 +85,5 @@
         </inertial>
     </link>
-	<!-- Camera properties
+	<!-- Camera properties -->
 	<joint name="camera_rgb_joint" type="fixed">
 		<parent link="head_tilt_link" />
@@ -131,6 +131,5 @@
         </inertial>
     </link>
-	-->
-	<!-- IMU properties -->
+	<!-- IMU properties
 	<joint name="imu_joint" type="fixed">
 		<parent link="base_link" />
@@ -147,5 +146,5 @@
                 izz="1.0" />
         </inertial>
-    </link>
+    </link>-->
 	<!-- Joint properties -->
 	<xacro:property name="joint_lower_limit" value="-${3.14}" />

Commit message: Remove pan from neck design

File: hexapod_description/urdf/phantomX_model.xacro (robot description, xacro)
@@ -50,5 +50,5 @@
         <material>Gazebo/DarkGrey</material>
     </gazebo>
-	<!-- Head Pan and Tilt properties -->
+	<!-- Head Pan and Tilt properties
 	<joint name="head_pan_joint" type="revolute">
 		<parent link="body_link"/>
@@ -67,7 +67,7 @@
                 izz="1.0" />
         </inertial>
-    </link>
+    </link> -->
 	<joint name="head_tilt_joint" type="revolute">
-		<parent link="head_pan_link"/>
+		<parent link="body_link"/>
 		<child link="head_tilt_link"/>
 		<axis xyz="0.0 1.0 0.0" />
@@ -131,5 +131,5 @@
         </inertial>
     </link>
-	<!-- IMU properties
+	<!-- IMU properties-->
 	<joint name="imu_joint" type="fixed">
 		<parent link="base_link" />
@@ -146,5 +146,5 @@
                 izz="1.0" />
         </inertial>
-    </link>-->
+    </link>
 	<!-- Joint properties -->
 	<xacro:property name="joint_lower_limit" value="-${3.14}" />

Commit message: startup changes

File: hexapod_description/urdf/phantomX_model.xacro (robot description, xacro)
@@ -50,5 +50,5 @@
         <material>Gazebo/DarkGrey</material>
     </gazebo>
-	<!-- Head Pan and Tilt properties
+	<!-- Head Pan and Tilt properties -->
 	<joint name="head_pan_joint" type="revolute">
 		<parent link="body_link"/>
@@ -67,7 +67,7 @@
                 izz="1.0" />
         </inertial>
-    </link> -->
+    </link>
 	<joint name="head_tilt_joint" type="revolute">
-		<parent link="body_link"/>
+		<parent link="head_pan_link"/>
 		<child link="head_tilt_link"/>
 		<axis xyz="0.0 1.0 0.0" />

Commit message: Your branch is up to date with 'origin/melodic_dev'.

File: hexapod_description/urdf/phantomX_model.xacro (robot description, xacro)
@@ -54,5 +54,5 @@
 		<parent link="body_link"/>
 		<child link="head_pan_link"/>
-		<axis xyz="0.0 0.0 1.0" />
+		<axis xyz="0.0 1.0 0.0" />
 		<origin xyz="0.145 0.0 0.080" />
 		<limit lower="-${3.14}" upper="${3.14}" effort="10000" velocity="100" />
